File: hardware/stargazer-motherboard/stargazer-motherboard.kicad_pcb (KiCad board)
At the start: 2 copper layers, 8 parts, among them J2_n1 swd-flywire, U1_n1 ADAFRUIT_FEATHER

Commit message: Now with thicc spaghetti
Parts:
- removed J2_n1: swd-flywire, Connector_PinHeader_2.54mm:PinHeader_1x02_P2.54mm_Vertical
- removed JP1_n1, JP5_n1: SolderJumper_2_Bridged, Jumper:SolderJumper-2_P1.3mm_Bridged_RoundedPad1.0x1.5mm
- removed JP2_n1, JP3_n1, JP4_n1: SolderJumper_2_Open, Jumper:SolderJumper-2_P1.3mm_Open_RoundedPad1.0x1.5mm
- added J?1: black-pill-leftovers, Connector_PinHeader_2.54mm:PinHeader_2x04_P2.54mm_Vertical, F.Cu at (71.1, 64.8)
- added U2_n1: SN74LVC125AD, Package_SO:SOIC-14_3.9x8.7mm_P1.27mm, F.Cu at (19.1, 55.9)
- moved U1_n1 14.9 mm to (36.8, 50.8), turned to 270 degrees
- moved U?1 4.56 mm to (47.0, 53.3), turned to 90 degrees
Connections:
- U?1 pad 38: /D9_n -> /D11_n
- U?1 pad 40: /D11_n -> /D9_n
Routing:
- net /BP6_n: track 0.00 -> 103.2 mm, vias 0 -> 4
- net /CARDn-CIPO: track 30.7 -> 98.4 mm
- net /D1_n: track 31.5 -> 77.0 mm, vias 1 -> 0
- net /BP5_n: track 0.00 -> 40.8 mm
- net /BP7_n: track 0.00 -> 33.8 mm, vias 0 -> 1
- net /CARDn-GO: track 28.6 -> 61.2 mm, vias 0 -> 2
- net /BP2_n: track 0.00 -> 29.4 mm
- net /VBATn: track 44.3 -> 17.3 mm, vias 0 -> 2
- net GND: track 76.1 -> 102.7 mm, vias 0 -> 1
- net /VBUSn: track 75.8 -> 49.5 mm
- net /CARDn-COPI: track 10.2 -> 36.5 mm, vias 0 -> 1
- net /BP8_n: track 0.00 -> 26.3 mm
- net /D0_n: track 26.5 -> 49.8 mm
- net /3v3_n: track 98.2 -> 75.1 mm, vias 1 -> 0
- net /BP4_n: track 0.00 -> 22.2 mm
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