File: hardware/backplane-feather-card/backplane-feather-card.kicad_pcb (KiCad board)
At the start: 2 copper layers, 117.5 x 58.4 mm, 31 parts, among them J1 card-header, J10 jumper, J11 jumper, J12 jumper, J13 card-programming-header-a, J14 card-programming-header-b, J2 jumper, J3 jumper, J5 jumper, J6 jumper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

Commit message: I dunno. working on v2 of the rack
Parts:
- R2, R3, R4, R5: value R -> 50 Ohm
