File: hardware/backplane-feather-card/backplane-feather-card.sch (KiCad schematic (older format))
At the start: 19 parts, among them J1 card-header, J13 card-programming-header-a, J14 card-programming-header-b, J2 jumper, J3 jumper, U1 ADAFRUIT_FEATHER, U5 SN74LVC125AD

Commit message: I dunno. working on v2 of the rack
Parts:
- R2, R3, R4, R5: value R -> 50 Ohm
Changed lines of the file:
@@
 P 4450 5450
 F 0 "R2" V 4243 5450 50  0000 C CNN
-F 1 "R" V 4334 5450 50  0000 C CNN
+F 1 "50 Ohm" V 4334 5450 50  0000 C CNN
 F 2 "Resistor_SMD:R_0805_2012Metric" V 4380 5450 50  0001 C CNN
 F 3 "~" H 4450 5450 50  0001 C CNN
@@
 P 4450 5750
 F 0 "R3" V 4243 5750 50  0000 C CNN
-F 1 "R" V 4334 5750 50  0000 C CNN
+F 1 "50 Ohm" V 4334 5750 50  0000 C CNN
 F 2 "Resistor_SMD:R_0805_2012Metric" V 4380 5750 50  0001 C CNN
 F 3 "~" H 4450 5750 50  0001 C CNN
@@
 P 4450 6050
 F 0 "R4" V 4243 6050 50  0000 C CNN
-F 1 "R" V 4334 6050 50  0000 C CNN
+F 1 "50 Ohm" V 4334 6050 50  0000 C CNN
 F 2 "Resistor_SMD:R_0805_2012Metric" V 4380 6050 50  0001 C CNN
 F 3 "~" H 4450 6050 50  0001 C CNN
@@
 P 4450 6350
 F 0 "R5" V 4243 6350 50  0000 C CNN
-F 1 "R" V 4334 6350 50  0000 C CNN
+F 1 "50 Ohm" V 4334 6350 50  0000 C CNN
 F 2 "Resistor_SMD:R_0805_2012Metric" V 4380 6350 50  0001 C CNN
 F 3 "~" H 4450 6350 50  0001 C CNN
