File: hardware/anachro-rack-module/anachro-rack-module.sch (KiCad schematic (older format))
At the start: 65 parts, among them J1 RACK-GPIO4, J10 RACK-UART, J11 RACK-GPIO4, J12 RACK-JTAG, J13 RACK-JTAG, J2 RACK-GPIO5, J3 8P8C, J4 8P8C, J5 RACK-POWER, J6 FPGA-A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

Commit message: Anachro test rack v2, plus fixed level shifter
Parts:
- added TP2, TP3: TestPoint, Connector_PinSocket_2.54mm:PinSocket_1x01_P2.54mm_Vertical, symbol Connector:TestPoint
Connections:
- net +3V3: now also Q1.1 (G)
- net +5V: now also TP3.1; no longer Q1.1 (G)
- net GND: now also TP2.1
- net ~FPGA-CRESET: no longer J6.5 (FPGA-CLK), JP9.1 (A)
- net FPGA-CDONE renamed ~FPGA-RST
- new net FPGA-CLK: J6.5 (FPGA-CLK), JP9.1 (A)
Changed lines of the file:
@@
 FPGA-COPI
 Text Label 2800 7500 2    50   ~ 0
-~FPGA-CRESET
+FPGA-CLK
 Text Label 5150 7150 2    50   ~ 0
 GPIO3
@@
 GPIO5
 Text Label 2800 7700 2    50   ~ 0
-FPGA-CDONE
+~FPGA-RST
 Text Label 2800 7600 2    50   ~ 0
 ~FPGA-IRQ
@@
 Text Label 5650 1100 2    50   ~ 0
 ~FPGA-CS
-Text Label 5650 1500 2    50   ~ 0
-~FPGA-CRESET
 Text Label 5650 2050 2    50   ~ 0
 ~FPGA-IRQ
-Text Label 5650 2150 2    50   ~ 0
-FPGA-CDONE
 Text Label 5650 1300 2    50   ~ 0
 FPGA-CIPO
@@
 NXP AN10441
 Wire Wire Line
-	7700 1200 7500 1200
-Wire Wire Line
-	7500 1200 7500 1400
-Connection ~ 7700 1200
-Wire Wire Line
 	7250 1700 7300 1700
 Connection ~ 7300 1700
@@
 Wire Wire Line
 	8950 2400 10050 2400
+Text Label 5650 1500 2    50   ~ 0
+FPGA-CLK
+Text Label 5650 2150 2    50   ~ 0
+~FPGA-RST
+$Comp
+L Connector:TestPoint TP2
+U 1 1 5FAA8618
+P 8300 2300
+F 0 "TP2" V 8400 2450 50  0000 C CNN
+F 1 "TestPoint" V 8200 2550 50  0000 C CNN
+F 2 "Connector_PinSocket_2.54mm:PinSocket_1x01_P2.54mm_Vertical" H 8500 2300 50  0001 C CNN
+F 3 "~" H 8500 2300 50  0001 C CNN
+	1    8300 2300
+	0    1    1    0
+$EndComp
+$Comp
+L Connector:TestPoint TP3
+U 1 1 5FAAFFFB
+P 8300 2600
+F 0 "TP3" V 8400 2750 50  0000 C CNN
+F 1 "TestPoint" V 8200 2850 50  0000 C CNN
+F 2 "Connector_PinSocket_2.54mm:PinSocket_1x01_P2.54mm_Vertical" H 8500 2600 50  0001 C CNN
+F 3 "~" H 8500 2600 50  0001 C CNN
+	1    8300 2600
+	0    1    1    0
+$EndComp
+$Comp
+L power:GND #PWR0137
+U 1 1 5FAB8A71
+P 8300 2300
+F 0 "#PWR0137" H 8300 2050 50  0001 C CNN
+F 1 "GND" H 8305 2127 50  0000 C CNN
+F 2 "" H 8300 2300 50  0001 C CNN
+F 3 "" H 8300 2300 50  0001 C CNN
+	1    8300 2300
+	0    1    1    0
+$EndComp
+$Comp
+L power:+5V #PWR0138
+U 1 1 5FAC2096
+P 8300 2600
+F 0 "#PWR0138" H 8300 2450 50  0001 C CNN
+F 1 "+5V" H 8315 2773 50  0000 C CNN
+F 2 "" H 8300 2600 50  0001 C CNN
+F 3 "" H 8300 2600 50  0001 C CNN
+	1    8300 2600
+	0    -1   -1   0
+$EndComp
+Wire Wire Line
+	7500 1400 7500 1200
+Wire Wire Line
+	7500 1200 7300 1200
+Connection ~ 7300 1200
 $EndSCHEMATC
